File: kicad/SAO-speaker-and-controller.kicad_pcb (KiCad board)
At the start: 2 copper layers, 28 x 28 mm, 18 parts, among them J1 SAO Connector, J2 SOICbite, U1 AT42QT1011-TSHR, U2 ATtiny85-20SU, U3 TPS613222ADBV

Commit message: Update design 4
Parts:
- D1: footprint Diode_SMD:D_0805_2012Metric -> Diode_SMD:D_SOD-323
Routing:
- net /~cs: track 18.4 -> 18.9 mm
